File: hw/address.sch (KiCad schematic (older format))
At the start: 8 parts

Commit message: updated schematic added footptints
Parts:
- R28, R29, R30, R31, R32, R33, R34, R35: footprint (none) -> Resistor_SMD:R_0805_2012Metric
Changed lines of the file:
@@
 F 0 "R28" H 3320 2846 50  0000 L CNN
 F 1 "10k" H 3320 2755 50  0000 L CNN
-F 2 "" V 3180 2800 50  0001 C CNN
+F 2 "Resistor_SMD:R_0805_2012Metric" V 3180 2800 50  0001 C CNN
 F 3 "~" H 3250 2800 50  0001 C CNN
 	1    3250 2800
@@
 F 0 "R29" H 3670 2846 50  0000 L CNN
 F 1 "10k" H 3670 2755 50  0000 L CNN
-F 2 "" V 3530 2800 50  0001 C CNN
+F 2 "Resistor_SMD:R_0805_2012Metric" V 3530 2800 50  0001 C CNN
 F 3 "~" H 3600 2800 50  0001 C CNN
 	1    3600 2800
@@
 F 0 "R30" H 4020 2846 50  0000 L CNN
 F 1 "10k" H 4020 2755 50  0000 L CNN
-F 2 "" V 3880 2800 50  0001 C CNN
+F 2 "Resistor_SMD:R_0805_2012Metric" V 3880 2800 50  0001 C CNN
 F 3 "~" H 3950 2800 50  0001 C CNN
 	1    3950 2800
@@
 F 0 "R31" H 4370 2846 50  0000 L CNN
 F 1 "10k" H 4370 2755 50  0000 L CNN
-F 2 "" V 4230 2800 50  0001 C CNN
+F 2 "Resistor_SMD:R_0805_2012Metric" V 4230 2800 50  0001 C CNN
 F 3 "~" H 4300 2800 50  0001 C CNN
 	1    4300 2800
@@
 F 0 "R32" H 4720 2846 50  0000 L CNN
 F 1 "10k" H 4720 2755 50  0000 L CNN
-F 2 "" V 4580 2800 50  0001 C CNN
+F 2 "Resistor_SMD:R_0805_2012Metric" V 4580 2800 50  0001 C CNN
 F 3 "~" H 4650 2800 50  0001 C CNN
 	1    4650 2800
@@
 F 0 "R33" H 5070 2846 50  0000 L CNN
 F 1 "10k" H 5070 2755 50  0000 L CNN
-F 2 "" V 4930 2800 50  0001 C CNN
+F 2 "Resistor_SMD:R_0805_2012Metric" V 4930 2800 50  0001 C CNN
 F 3 "~" H 5000 2800 50  0001 C CNN
 	1    5000 2800
@@
 F 0 "R34" H 5420 2846 50  0000 L CNN
 F 1 "10k" H 5420 2755 50  0000 L CNN
-F 2 "" V 5280 2800 50  0001 C CNN
+F 2 "Resistor_SMD:R_0805_2012Metric" V 5280 2800 50  0001 C CNN
 F 3 "~" H 5350 2800 50  0001 C CNN
 	1    5350 2800
@@
 F 0 "R35" H 5770 2846 50  0000 L CNN
 F 1 "10k" H 5770 2755 50  0000 L CNN
-F 2 "" V 5630 2800 50  0001 C CNN
+F 2 "Resistor_SMD:R_0805_2012Metric" V 5630 2800 50  0001 C CNN
 F 3 "~" H 5700 2800 50  0001 C CNN
 	1    5700 2800
