File: hw/ir.sch (KiCad schematic (older format))
At the start: 3 parts, among them U12 OSRB38C9BA

Commit message: updated schematic added footptints
Parts:
- R27: footprint Resistor_SMD:R_0805_2012Metric_Pad1.15x1.50mm_HandSolder -> Resistor_SMD:R_0805_2012Metric
Changed lines of the file:
@@
 F 0 "R27" H 4070 2196 50  0000 L CNN
 F 1 "100R" H 4070 2105 50  0000 L CNN
-F 2 "Resistor_SMD:R_0805_2012Metric_Pad1.15x1.50mm_HandSolder" V 3930 2150 50  0001 C CNN
+F 2 "Resistor_SMD:R_0805_2012Metric" V 3930 2150 50  0001 C CNN
 F 3 "" H 4000 2150 50  0001 C CNN
 	1    4000 2150

Commit message: updated schematic
Parts:
- removed U12: OSRB38C9BA, KLIB_Opto:OSRB8C9BA, symbol KLIB_Opto:OSRB38C9BA
- added U11: OSRB38C9BA, KLIB_Opto:OSRB8C9BA_Horizontal, symbol KLIB_Opto:OSRB38C9BA
Connections:
- net GND: now also U11.2 (GND)
- net IR_RX: now also U11.1 (OUT)
- net at C35.1, R27.2: now also U11.3 (VCC)
Changed lines of the file:
@@
 $EndDescr
-$Comp
-L KLIB_Opto:OSRB38C9BA U12
-U 1 1 5ACFE558
-P 3500 2450
-F 0 "U12" H 3476 2817 50  0000 C CNN
-F 1 "OSRB38C9BA" H 3476 2726 50  0000 C CNN
-F 2 "KLIB_Opto:OSRB8C9BA" H 3300 2600 10  0001 C CNN
-F 3 "http://www.tme.eu/cz/Document/777fdf21e0fba3fd5c036ef95756460c/OSRB38C9BA.pdf" H 3550 2100 50  0001 C CNN
-	1    3500 2450
-	1    0    0    -1
-$EndComp
 $Comp
 L Device:CP C35
@@
 $EndComp
 $Comp
-L KLIB_Power:GND #PWR083
+L KLIB_Power:GND #PWR082
 U 1 1 5ACFE566
 P 4000 2800
-F 0 "#PWR083" H 4000 2600 50  0001 C CNN
+F 0 "#PWR082" H 4000 2600 50  0001 C CNN
 F 1 "GND" H 4005 2627 50  0000 C CNN
 F 2 "" H 4000 2800 50  0001 C CNN
@@
 $EndComp
 $Comp
-L KLIB_Power:GND #PWR081
+L KLIB_Power:GND #PWR080
 U 1 1 5ACFE56C
 P 3800 2800
-F 0 "#PWR081" H 3800 2600 50  0001 C CNN
+F 0 "#PWR080" H 3800 2600 50  0001 C CNN
 F 1 "GND" H 3805 2627 50  0000 C CNN
 F 2 "" H 3800 2800 50  0001 C CNN
@@
 $EndComp
 $Comp
-L KLIB_Power:+5V #PWR082
+L KLIB_Power:+5V #PWR081
 U 1 1 5ACFE572
 P 4000 2000
-F 0 "#PWR082" H 4000 1700 50  0001 C CNN
+F 0 "#PWR081" H 4000 1700 50  0001 C CNN
 F 1 "+5V" H 4005 2173 50  0000 C CNN
 F 2 "" H 4000 2000 50  0001 C CNN
@@
 IR_RX
 $Comp
-L KLIB_Power:PWR_FLAG #FLG05
+L KLIB_Power:PWR_FLAG #FLG07
 U 1 1 5ACFE586
 P 4000 2350
-F 0 "#FLG05" H 4000 2425 50  0001 C CNN
+F 0 "#FLG07" H 4000 2425 50  0001 C CNN
 F 1 "PWR_FLAG" V 4000 2478 50  0000 L CNN
 F 2 "" H 4000 2350 50  0001 C CNN
@@
 Wire Wire Line
 	3800 2450 4950 2450
+$Comp
+L KLIB_Opto:OSRB38C9BA U11
+U 1 1 5AD823E6
+P 3500 2450
+F 0 "U11" H 3476 2817 50  0000 C CNN
+F 1 "OSRB38C9BA" H 3476 2726 50  0000 C CNN
+F 2 "KLIB_Opto:OSRB8C9BA_Horizontal" H 3500 2100 50  0001 C CNN
+F 3 "http://www.tme.eu/cz/Document/777fdf21e0fba3fd5c036ef95756460c/OSRB38C9BA.pdf" H 3550 2100 50  0001 C CNN
+	1    3500 2450
+	1    0    0    -1
+$EndComp
 $EndSCHEMATC
