File: hw/led.sch (KiCad schematic (older format))
At the start: 17 parts, among them U9 ULN2003

Commit message: updated schematic added footptints
Parts:
- R15, R16, R17, R18, R19, R20, R21, R22, R23, R24, R25, R26: footprint (none) -> Resistor_SMD:R_0805_2012Metric
- U9: footprint (none) -> Package_SO:SOIC-16_3.9x9.9mm_P1.27mm
Changed lines of the file:
@@
 F 0 "U9" H 2650 4767 50  0000 C CNN
 F 1 "ULN2003" H 2650 4676 50  0000 C CNN
-F 2 "" H 2700 3550 50  0001 L CNN
+F 2 "Package_SO:SOIC-16_3.9x9.9mm_P1.27mm" H 2700 3550 50  0001 L CNN
 F 3 "http://www.ti.com/lit/ds/symlink/uln2003a.pdf" H 2750 3900 50  0001 C CNN
 	1    2650 4100
@@
 F 0 "R17" H 4170 3696 50  0000 L CNN
 F 1 "180R" H 4170 3605 50  0000 L CNN
-F 2 "" V 4030 3650 50  0001 C CNN
+F 2 "Resistor_SMD:R_0805_2012Metric" V 4030 3650 50  0001 C CNN
 F 3 "~" H 4100 3650 50  0001 C CNN
 	1    4100 3650
@@
 F 0 "R16" H 3820 3696 50  0000 L CNN
 F 1 "120R" H 3820 3605 50  0000 L CNN
-F 2 "" V 3680 3650 50  0001 C CNN
+F 2 "Resistor_SMD:R_0805_2012Metric" V 3680 3650 50  0001 C CNN
 F 3 "~" H 3750 3650 50  0001 C CNN
 	1    3750 3650
@@
 F 0 "R15" H 3470 3696 50  0000 L CNN
 F 1 "120R" H 3470 3605 50  0000 L CNN
-F 2 "" V 3330 3650 50  0001 C CNN
+F 2 "Resistor_SMD:R_0805_2012Metric" V 3330 3650 50  0001 C CNN
 F 3 "~" H 3400 3650 50  0001 C CNN
 	1    3400 3650
@@
 F 0 "R20" H 5970 3696 50  0000 L CNN
 F 1 "180R" H 5970 3605 50  0000 L CNN
-F 2 "" V 5830 3650 50  0001 C CNN
+F 2 "Resistor_SMD:R_0805_2012Metric" V 5830 3650 50  0001 C CNN
 F 3 "~" H 5900 3650 50  0001 C CNN
 	1    5900 3650
@@
 F 0 "R19" H 5620 3696 50  0000 L CNN
 F 1 "120R" H 5620 3605 50  0000 L CNN
-F 2 "" V 5480 3650 50  0001 C CNN
+F 2 "Resistor_SMD:R_0805_2012Metric" V 5480 3650 50  0001 C CNN
 F 3 "~" H 5550 3650 50  0001 C CNN
 	1    5550 3650
@@
 F 0 "R18" H 5270 3696 50  0000 L CNN
 F 1 "120R" H 5270 3605 50  0000 L CNN
-F 2 "" V 5130 3650 50  0001 C CNN
+F 2 "Resistor_SMD:R_0805_2012Metric" V 5130 3650 50  0001 C CNN
 F 3 "~" H 5200 3650 50  0001 C CNN
 	1    5200 3650
@@
 F 0 "R23" H 7770 3696 50  0000 L CNN
 F 1 "180R" H 7770 3605 50  0000 L CNN
-F 2 "" V 7630 3650 50  0001 C CNN
+F 2 "Resistor_SMD:R_0805_2012Metric" V 7630 3650 50  0001 C CNN
 F 3 "~" H 7700 3650 50  0001 C CNN
 	1    7700 3650
@@
 F 0 "R22" H 7420 3696 50  0000 L CNN
 F 1 "120R" H 7420 3605 50  0000 L CNN
-F 2 "" V 7280 3650 50  0001 C CNN
+F 2 "Resistor_SMD:R_0805_2012Metric" V 7280 3650 50  0001 C CNN
 F 3 "~" H 7350 3650 50  0001 C CNN
 	1    7350 3650
@@
 F 0 "R21" H 7070 3696 50  0000 L CNN
 F 1 "120R" H 7070 3605 50  0000 L CNN
-F 2 "" V 6930 3650 50  0001 C CNN
+F 2 "Resistor_SMD:R_0805_2012Metric" V 6930 3650 50  0001 C CNN
 F 3 "~" H 7000 3650 50  0001 C CNN
 	1    7000 3650
@@
 F 0 "R26" H 9570 3696 50  0000 L CNN
 F 1 "180R" H 9570 3605 50  0000 L CNN
-F 2 "" V 9430 3650 50  0001 C CNN
+F 2 "Resistor_SMD:R_0805_2012Metric" V 9430 3650 50  0001 C CNN
 F 3 "~" H 9500 3650 50  0001 C CNN
 	1    9500 3650
@@
 F 0 "R25" H 9220 3696 50  0000 L CNN
 F 1 "120R" H 9220 3605 50  0000 L CNN
-F 2 "" V 9080 3650 50  0001 C CNN
+F 2 "Resistor_SMD:R_0805_2012Metric" V 9080 3650 50  0001 C CNN
 F 3 "~" H 9150 3650 50  0001 C CNN
 	1    9150 3650
@@
 F 0 "R24" H 8870 3696 50  0000 L CNN
 F 1 "120R" H 8870 3605 50  0000 L CNN
-F 2 "" V 8730 3650 50  0001 C CNN
+F 2 "Resistor_SMD:R_0805_2012Metric" V 8730 3650 50  0001 C CNN
 F 3 "~" H 8800 3650 50  0001 C CNN
 	1    8800 3650

Commit message: updated schematic
Parts:
- D2, D3, D4, D5: footprint LEDs:LED_WS2812-PLCC6 -> KLIB_Opto:LED_RGB_5050-6
- renumbered U9 to U8
