File: hw/sound.sch (KiCad schematic (older format))
At the start: 27 parts

Commit message: finished schematic
Parts:
- gave numbers to parts that had none: 24
Connections:
- net sheet5AEA7AF2/DAC renamed Sound MCU/DAC

Commit message: updated schematic added footptints
Parts:
- C10, C11, C12, C13, C14, C15, C16, C17, C9: footprint (none) -> Capacitor_SMD:C_0805_2012Metric
- R10, R11, R12, R3, R4, R5, R6, R7, R8, R9: footprint (none) -> Resistor_SMD:R_0805_2012Metric
Changed lines of the file:
@@
 F 0 "R9" V 5043 1750 50  0000 C CNN
 F 1 "18k" V 5134 1750 50  0000 C CNN
-F 2 "" V 5180 1750 50  0001 C CNN
+F 2 "Resistor_SMD:R_0805_2012Metric" V 5180 1750 50  0001 C CNN
 F 3 "~" H 5250 1750 50  0001 C CNN
 	1    5250 1750
@@
 F 0 "R10" V 5443 1750 50  0000 C CNN
 F 1 "470k" V 5534 1750 50  0000 C CNN
-F 2 "" V 5580 1750 50  0001 C CNN
+F 2 "Resistor_SMD:R_0805_2012Metric" V 5580 1750 50  0001 C CNN
 F 3 "~" H 5650 1750 50  0001 C CNN
 	1    5650 1750
@@
 F 0 "C12" V 6302 1250 50  0000 C CNN
 F 1 "1n" V 6211 1250 50  0000 C CNN
-F 2 "" H 6088 1100 50  0001 C CNN
+F 2 "Capacitor_SMD:C_0805_2012Metric" H 6088 1100 50  0001 C CNN
 F 3 "~" H 6050 1250 50  0001 C CNN
 	1    6050 1250
@@
 F 0 "C11" H 5965 2246 50  0000 L CNN
 F 1 "100p" H 5965 2155 50  0000 L CNN
-F 2 "" H 5888 2050 50  0001 C CNN
+F 2 "Capacitor_SMD:C_0805_2012Metric" H 5888 2050 50  0001 C CNN
 F 3 "~" H 5850 2200 50  0001 C CNN
 	1    5850 2200
@@
 F 0 "R11" V 6893 1850 50  0000 C CNN
 F 1 "82k" V 6984 1850 50  0000 C CNN
-F 2 "" V 7030 1850 50  0001 C CNN
+F 2 "Resistor_SMD:R_0805_2012Metric" V 7030 1850 50  0001 C CNN
 F 3 "~" H 7100 1850 50  0001 C CNN
 	1    7100 1850
@@
 F 0 "R12" V 7293 1850 50  0000 C CNN
 F 1 "82k" V 7384 1850 50  0000 C CNN
-F 2 "" V 7430 1850 50  0001 C CNN
+F 2 "Resistor_SMD:R_0805_2012Metric" V 7430 1850 50  0001 C CNN
 F 3 "~" H 7500 1850 50  0001 C CNN
 	1    7500 1850
@@
 F 0 "C15" V 8152 1350 50  0000 C CNN
 F 1 "1n" V 8061 1350 50  0000 C CNN
-F 2 "" H 7938 1200 50  0001 C CNN
+F 2 "Capacitor_SMD:C_0805_2012Metric" H 7938 1200 50  0001 C CNN
 F 3 "~" H 7900 1350 50  0001 C CNN
 	1    7900 1350
@@
 F 0 "C13" H 7815 2346 50  0000 L CNN
 F 1 "68p" H 7815 2255 50  0000 L CNN
-F 2 "" H 7738 2150 50  0001 C CNN
+F 2 "Capacitor_SMD:C_0805_2012Metric" H 7738 2150 50  0001 C CNN
 F 3 "~" H 7700 2300 50  0001 C CNN
 	1    7700 2300
@@
 F 0 "R5" H 4070 1346 50  0000 L CNN
 F 1 "R" H 4070 1255 50  0000 L CNN
-F 2 "" V 3930 1300 50  0001 C CNN
+F 2 "Resistor_SMD:R_0805_2012Metric" V 3930 1300 50  0001 C CNN
 F 3 "~" H 4000 1300 50  0001 C CNN
 	1    4000 1300
@@
 F 0 "R6" H 4070 2146 50  0000 L CNN
 F 1 "R" H 4070 2055 50  0000 L CNN
-F 2 "" V 3930 2100 50  0001 C CNN
+F 2 "Resistor_SMD:R_0805_2012Metric" V 3930 2100 50  0001 C CNN
 F 3 "~" H 4000 2100 50  0001 C CNN
 	1    4000 2100
@@
 F 0 "C17" V 9698 2050 50  0000 C CNN
 F 1 "1u/50V" V 9789 2050 50  0000 C CNN
-F 2 "" H 9988 1900 50  0001 C CNN
+F 2 "Capacitor_SMD:C_0805_2012Metric" H 9988 1900 50  0001 C CNN
 F 3 "~" H 9950 2050 50  0001 C CNN
 	1    9950 2050
@@
 F 0 "C9" H 2465 5246 50  0000 L CNN
 F 1 "1u/50V" H 2465 5155 50  0000 L CNN
-F 2 "" H 2388 5050 50  0001 C CNN
+F 2 "Capacitor_SMD:C_0805_2012Metric" H 2388 5050 50  0001 C CNN
 F 3 "~" H 2350 5200 50  0001 C CNN
 	1    2350 5200
@@
 F 0 "R3" V 1943 4150 50  0000 C CNN
 F 1 "10k" V 2034 4150 50  0000 C CNN
-F 2 "" V 2080 4150 50  0001 C CNN
+F 2 "Resistor_SMD:R_0805_2012Metric" V 2080 4150 50  0001 C CNN
 F 3 "~" H 2150 4150 50  0001 C CNN
 	1    2150 4150
@@
 F 0 "R4" V 2693 3400 50  0000 C CNN
 F 1 "10k" V 2784 3400 50  0000 C CNN
-F 2 "" V 2830 3400 50  0001 C CNN
+F 2 "Resistor_SMD:R_0805_2012Metric" V 2830 3400 50  0001 C CNN
 F 3 "~" H 2900 3400 50  0001 C CNN
 	1    2900 3400
@@
 F 0 "C10" H 4665 6946 50  0000 L CNN
 F 1 "1u/50V" H 4665 6855 50  0000 L CNN
-F 2 "" H 4588 6750 50  0001 C CNN
+F 2 "Capacitor_SMD:C_0805_2012Metric" H 4588 6750 50  0001 C CNN
 F 3 "~" H 4550 6900 50  0001 C CNN
 	1    4550 6900
@@
 F 0 "R7" V 4143 5850 50  0000 C CNN
 F 1 "10k" V 4234 5850 50  0000 C CNN
-F 2 "" V 4280 5850 50  0001 C CNN
+F 2 "Resistor_SMD:R_0805_2012Metric" V 4280 5850 50  0001 C CNN
 F 3 "~" H 4350 5850 50  0001 C CNN
 	1    4350 5850
@@
 F 0 "R8" V 4893 5100 50  0000 C CNN
 F 1 "10k" V 4984 5100 50  0000 C CNN
-F 2 "" V 5030 5100 50  0001 C CNN
+F 2 "Resistor_SMD:R_0805_2012Metric" V 5030 5100 50  0001 C CNN
 F 3 "~" H 5100 5100 50  0001 C CNN
 	1    5100 5100
@@
 F 0 "C14" H 7965 4796 50  0000 L CNN
 F 1 "100n" H 7965 4705 50  0000 L CNN
-F 2 "" H 7888 4600 50  0001 C CNN
+F 2 "Capacitor_SMD:C_0805_2012Metric" H 7888 4600 50  0001 C CNN
 F 3 "~" H 7850 4750 50  0001 C CNN
 	1    7850 4750
@@
 F 0 "C16" H 9515 4796 50  0000 L CNN
 F 1 "100n" H 9515 4705 50  0000 L CNN
-F 2 "" H 9438 4600 50  0001 C CNN
+F 2 "Capacitor_SMD:C_0805_2012Metric" H 9438 4600 50  0001 C CNN
 F 3 "~" H 9400 4750 50  0001 C CNN
 	1    9400 4750

Commit message: updated schematic
Parts:
- renumbered U5 to U3, U3 to U5, U6 to U5
Connections:
- net at C12.2, R11.2: now also U3.6 (-), U3.7; no longer U3.1, U3.2 (-)
- net at C11.1, R10.1: now also U3.5 (+); no longer U3.3 (+)
- net at C13.1, R12.1: now also U5.3 (+); no longer U5.5 (+)
- new net: C15.2, U5.1, U5.2 (-), U5.5 (+)
- new net: C17.2, U5.6 (-), U5.7
Changed lines of the file:
@@
 	1500 1550 2250 1550
 $Comp
-L KLIB_Audio:AD8542 U5
-U 1 1 5ACD4FF8
+L KLIB_Audio:AD8542 U3
+U 2 1 5ACD4FF8
 P 6550 1850
-F 0 "U5" H 6550 2285 50  0000 C CNN
+F 0 "U3" H 6550 2285 50  0000 C CNN
 F 1 "AD8542" H 6550 2194 50  0000 C CNN
 F 2 "Package_SO:SOIJ-8_5.3x5.3mm_P1.27mm" H 6750 1650 50  0001 L CNN
 F 3 "http://www.analog.com/media/en/technical-documentation/data-sheets/AD8541_8542_8544.pdf" H 6700 2000 50  0001 C CNN
-	1    6550 1850
+	2    6550 1850
 	1    0    0    -1
 $EndComp
@@
 	5450 1750 5400 1750
 $Comp
-L KLIB_Audio:AD8542 U3
-U 2 1 5ACD61E9
+L KLIB_Audio:AD8542 U5
+U 1 1 5ACD61E9
 P 8400 1950
-F 0 "U3" H 8400 2385 50  0000 C CNN
+F 0 "U5" H 8400 2385 50  0000 C CNN
 F 1 "AD8542" H 8400 2294 50  0000 C CNN
 F 2 "Package_SO:SOIJ-8_5.3x5.3mm_P1.27mm" H 8600 1750 50  0001 L CNN
 F 3 "http://www.analog.com/media/en/technical-documentation/data-sheets/AD8541_8542_8544.pdf" H 8550 2100 50  0001 C CNN
-	2    8400 1950
+	1    8400 1950
 	1    0    0    -1
 $EndComp
@@
 	8750 1950 9100 1950
 $Comp
-L KLIB_Audio:AD8542 U6
-U 1 1 5ACE046E
+L KLIB_Audio:AD8542 U5
+U 2 1 5ACE046E
 P 9400 2050
-F 0 "U6" H 9400 2485 50  0000 C CNN
+F 0 "U5" H 9400 2485 50  0000 C CNN
 F 1 "AD8542" H 9400 2394 50  0000 C CNN
 F 2 "Package_SO:SOIJ-8_5.3x5.3mm_P1.27mm" H 9600 1850 50  0001 L CNN
 F 3 "http://www.analog.com/media/en/technical-documentation/data-sheets/AD8541_8542_8544.pdf" H 9550 2200 50  0001 C CNN
-	1    9400 2050
-	1    0    0    -1
-$EndComp
+	2    9400 2050
+	1    0    0    -1
+$EndComp
