File: hw/sound_mcu.sch (KiCad schematic (older format))
At the start: 12 parts, among them J4 SWD_01X04, U5 STM32F405RGTx

Commit message: finished schematic
Parts:
- removed C10, C12, C13, C15, C16: 100n, symbol Device:C
- removed J4: SWD_01X04, Connector_PinHeader_2.54mm:PinHeader_1x04_P2.54mm_Vertical, symbol KLIB_Connector_Prog:SWD_01X04
- removed U5: STM32F405RGTx, LQFP64, symbol MCU_ST_STM32:STM32F405RGTx
- added C18, C20, C21, C23, C24: 100n, symbol Device:C
- added J3: SWD_01X04, Connector_PinHeader_2.54mm:PinHeader_1x04_P2.54mm_Vertical, symbol KLIB_Connector_Prog:SWD_01X04
- added U7: STM32F405RGTx, LQFP64, symbol MCU_ST_STM32:STM32F405RGTx
- renumbered C11 to C19, C14 to C22, C17 to C25, R11 to R13, R12 to R14
Connections:
- net +3V3: now also C20.1, C21.1, C23.1, C24.1, U7.1 (VBAT), U7.13 (VDDA), U7.19 (VDD), U7.32 (VDD), U7.48 (VDD), U7.64 (VDD)
- net DAC: now also U7.20 (ADC1_IN4/ADC2_IN4/DAC_OUT1/I2S3_WS/SPI1_NSS/SPI3_NSS/USART2_CK/USB_OTG_HS_SOF/PA4)
- net GND: now also C18.2, C20.2, C21.2, C23.2, C24.2, J3.1 (GND), U7.12 (VSSA), U7.18 (VSS), U7.63 (VSS)
- net MUTE: now also U7.22 (ADC1_IN6/ADC2_IN6/SPI1_MISO/TIM13_CH1/TIM1_BKIN/TIM3_CH1/TIM8_BKIN/PA6)
- net SOUND_SEL0: now also U7.14 (ADC1_IN0/ADC2_IN0/ADC3_IN0/SYS_WKUP/TIM2_CH1/TIM2_ETR/TIM5_CH1/TIM8_ETR/UART4_TX/USART2_CTS/PA0)
- net SOUND_SEL1: now also U7.15 (ADC1_IN1/ADC2_IN1/ADC3_IN1/TIM2_CH2/TIM5_CH2/UART4_RX/USART2_RTS/PA1)
- net SOUND_UART_RX: now also U7.43 (TIM1_CH3/USART1_RX/USB_OTG_FS_ID/PA10)
- net SOUND_UART_TX: now also U7.42 (DAC_EXTI9/I2C3_SMBA/TIM1_CH2/USART1_TX/USB_OTG_FS_VBUS/PA9)
- net SWDCLK: now also J3.3 (SWCLK), U7.49 (SYS_JTCK-SWCLK/PA14)
- net SWDIO: now also J3.4 (SWDIO), U7.46 (SYS_JTMS-SWDIO/PA13)
- net ~RST: now also J3.2 (~RST), U7.7 (NRST)
- net at C19.1: now also U7.47 (VCAP_2)
- net at R13.2: now also U7.60 (BOOT0)
- new net: C18.1, U7.31 (VCAP_1)
Changed lines of the file:
@@
 $Descr A4 11693 8268
 encoding utf-8
-Sheet 4 4
-Title "microcontroller for sound generator"
+Sheet 4 14
+Title "MCU for sound generator"
 Date "2018-04-10"
 Rev "1.0"
@@
 $EndDescr
 $Comp
-L MCU_ST_STM32:STM32F405RGTx U5
-U 1 1 5ACE8377
+L MCU_ST_STM32:STM32F405RGTx U7
+U 1 1 5AD7FB27
 P 5850 3750
-F 0 "U5" H 1650 5850 50  0000 L CNN
+F 0 "U7" H 1650 5850 50  0000 L CNN
 F 1 "STM32F405RGTx" H 1650 5750 50  0000 L CNN
 F 2 "LQFP64" H 10050 5625 50  0001 R TNN
@@
 $EndComp
 $Comp
-L KLIB_Power:+3V3 #PWR038
+L KLIB_Power:+3V3 #PWR031
 U 1 1 5ACE8468
 P 5850 1650
-F 0 "#PWR038" H 5850 1350 50  0001 C CNN
+F 0 "#PWR031" H 5850 1350 50  0001 C CNN
 F 1 "+3V3" H 5855 1823 50  0000 C CNN
 F 2 "" H 5850 1650 50  0001 C CNN
@@
 	5950 1700 6050 1700
 $Comp
-L KLIB_Power:GND #PWR039
+L KLIB_Power:GND #PWR032
 U 1 1 5ACE8945
 P 5850 5850
-F 0 "#PWR039" H 5850 5650 50  0001 C CNN
+F 0 "#PWR032" H 5850 5650 50  0001 C CNN
 F 1 "GND" H 5855 5677 50  0000 C CNN
 F 2 "" H 5850 5850 50  0001 C CNN
@@
 	5750 5800 5750 5750
 $Comp
-L Device:R R12
+L Device:R R14
 U 1 1 5ACE9349
 P 1100 1950
-F 0 "R12" H 1170 1996 50  0000 L CNN
+F 0 "R14" H 1170 1996 50  0000 L CNN
 F 1 "10k" H 1170 1905 50  0000 L CNN
 F 2 "" V 1030 1950 50  0001 C CNN
@@
 	1100 2150 1100 2100
 $Comp
-L Device:R R11
+L Device:R R13
 U 1 1 5ACE9526
 P 750 1950
-F 0 "R11" H 820 1996 50  0000 L CNN
+F 0 "R13" H 820 1996 50  0000 L CNN
 F 1 "10k" H 820 1905 50  0000 L CNN
 F 2 "" V 680 1950 50  0001 C CNN
@@
 $EndComp
 $Comp
-L KLIB_Power:GND #PWR032
+L KLIB_Power:GND #PWR026
 U 1 1 5ACE95CC
 P 750 1700
-F 0 "#PWR032" H 750 1500 50  0001 C CNN
+F 0 "#PWR026" H 750 1500 50  0001 C CNN
 F 1 "GND" H 755 1527 50  0000 C CNN
 F 2 "" H 750 1700 50  0001 C CNN
@@
 $EndComp
 $Comp
-L KLIB_Power:+3V3 #PWR034
+L KLIB_Power:+3V3 #PWR028
 U 1 1 5ACE967B
 P 1100 1700
-F 0 "#PWR034" H 1100 1400 50  0001 C CNN
+F 0 "#PWR028" H 1100 1400 50  0001 C CNN
 F 1 "+3V3" H 1105 1873 50  0000 C CNN
 F 2 "" H 1100 1700 50  0001 C CNN
@@
 SOUND_UART_TX
 $Comp
-L KLIB_Connector_Prog:SWD_01X04 J4
-U 1 1 5ACF9C1C
+L KLIB_Connector_Prog:SWD_01X04 J3
+U 1 1 5AD7FB2E
 P 5650 7100
-F 0 "J4" H 5370 7196 50  0000 R CNN
+F 0 "J3" H 5370 7196 50  0000 R CNN
 F 1 "SWD_01X04" H 5370 7105 50  0000 R CNN
 F 2 "Connector_PinHeader_2.54mm:PinHeader_1x04_P2.54mm_Vertical" H 5600 6700 50  0001 C CNN
@@
 	5450 7100 5000 7100
 $Comp
-L KLIB_Power:GND #PWR037
+L KLIB_Power:GND #PWR030
 U 1 1 5ACFAB32
 P 5450 7200
-F 0 "#PWR037" H 5450 7000 50  0001 C CNN
+F 0 "#PWR030" H 5450 7000 50  0001 C CNN
 F 1 "GND" H 5455 7027 50  0000 C CNN
 F 2 "" H 5450 7200 50  0001 C CNN
@@
 NoConn ~ 1550 3350
 $Comp
-L Device:C C10
-U 1 1 5AD22BDE
+L Device:C C18
+U 1 1 5AD7FB30
 P 750 2950
-F 0 "C10" H 865 2996 50  0000 L CNN
+F 0 "C18" H 865 2996 50  0000 L CNN
 F 1 "100n" H 865 2905 50  0000 L CNN
 F 2 "" H 788 2800 50  0001 C CNN
@@
 $EndComp
 $Comp
-L Device:C C11
+L Device:C C19
 U 1 1 5AD22C3E
 P 1250 2950
-F 0 "C11" H 1365 2996 50  0000 L CNN
+F 0 "C19" H 1365 2996 50  0000 L CNN
 F 1 "100n" H 1365 2905 50  0000 L CNN
 F 2 "" H 1288 2800 50  0001 C CNN
@@
 $EndComp
 $Comp
-L KLIB_Power:GND #PWR035
+L KLIB_Power:GND #PWR029
 U 1 1 5AD22D21
 P 1250 3100
-F 0 "#PWR035" H 1250 2900 50  0001 C CNN
+F 0 "#PWR029" H 1250 2900 50  0001 C CNN
 F 1 "GND" H 1255 2927 50  0000 C CNN
 F 2 "" H 1250 3100 50  0001 C CNN
@@
 $EndComp
 $Comp
-L KLIB_Power:GND #PWR033
+L KLIB_Power:GND #PWR027
 U 1 1 5AD22D74
 P 750 3100
-F 0 "#PWR033" H 750 2900 50  0001 C CNN
+F 0 "#PWR027" H 750 2900 50  0001 C CNN
 F 1 "GND" H 755 2927 50  0000 C CNN
 F 2 "" H 750 3100 50  0001 C CNN
@@
 	1250 2750 1250 2800
 $Comp
-L Device:C C13
-U 1 1 5AD26339
+L Device:C C21
+U 1 1 5AD7FB34
 P 7750 1150
-F 0 "C13" H 7865 1196 50  0000 L CNN
+F 0 "C21" H 7865 1196 50  0000 L CNN
 F 1 "100n" H 7865 1105 50  0000 L CNN
 F 2 "" H 7788 1000 50  0001 C CNN
@@
 $EndComp
 $Comp
-L Device:C C14
+L Device:C C22
 U 1 1 5AD26340
 P 8200 1150
-F 0 "C14" H 8315 1196 50  0000 L CNN
+F 0 "C22" H 8315 1196 50  0000 L CNN
 F 1 "100n" H 8315 1105 50  0000 L CNN
 F 2 "" H 8238 1000 50  0001 C CNN
@@
 $EndComp
 $Comp
-L Device:C C15
-U 1 1 5AD26347
+L Device:C C23
+U 1 1 5AD7FB36
 P 8650 1150
-F 0 "C15" H 8765 1196 50  0000 L CNN
+F 0 "C23" H 8765 1196 50  0000 L CNN
 F 1 "100n" H 8765 1105 50  0000 L CNN
 F 2 "" H 8688 1000 50  0001 C CNN
@@
 $EndComp
 $Comp
-L Device:C C16
-U 1 1 5AD2634E
+L Device:C C24
+U 1 1 5AD7FB37
 P 9100 1150
-F 0 "C16" H 9215 1196 50  0000 L CNN
+F 0 "C24" H 9215 1196 50  0000 L CNN
 F 1 "100n" H 9215 1105 50  0000 L CNN
 F 2 "" H 9138 1000 50  0001 C CNN
@@
 $EndComp
 $Comp
-L Device:C C17
+L Device:C C25
 U 1 1 5AD26355
 P 9550 1150
-F 0 "C17" H 9665 1196 50  0000 L CNN
+F 0 "C25" H 9665 1196 50  0000 L CNN
 F 1 "100n" H 9665 1105 50  0000 L CNN
 F 2 "" H 9588 1000 50  0001 C CNN
@@
 $EndComp
 $Comp
-L Device:C C12
-U 1 1 5AD2636A
+L Device:C C20
+U 1 1 5AD7FB39
 P 7300 1150
-F 0 "C12" H 7415 1196 50  0000 L CNN
+F 0 "C20" H 7415 1196 50  0000 L CNN
 F 1 "100n" H 7415 1105 50  0000 L CNN
 F 2 "" H 7338 1000 50  0001 C CNN
@@
 	9550 1000 9550 950
 $Comp
-L KLIB_Power:+3V3 #PWR040
-U 1 1 5AD26399
+L KLIB_Power:+3V3 #PWR033
+U 1 1 5AD7FB3A
 P 8450 900
-F 0 "#PWR040" H 8450 600 50  0001 C CNN
+F 0 "#PWR033" H 8450 600 50  0001 C CNN
 F 1 "+3V3" H 8455 1073 50  0000 C CNN
 F 2 "" H 8450 900 50  0001 C CNN
@@
 $EndComp
 $Comp
-L KLIB_Power:GND #PWR041
-U 1 1 5AD2639F
+L KLIB_Power:GND #PWR034
+U 1 1 5AD7FB3B
 P 8450 1400
-F 0 "#PWR041" H 8450 1200 50  0001 C CNN
+F 0 "#PWR034" H 8450 1200 50  0001 C CNN
 F 1 "GND" H 8455 1227 50  0000 C CNN
 F 2 "" H 8450 1400 50  0001 C CNN
@@
 	8450 950  8650 950
 $Comp
-L KLIB_Power:PWR_FLAG #FLG0101
-U 1 1 5AE70DE3
+L KLIB_Power:PWR_FLAG #FLG03
+U 1 1 5AD7FB3C
 P 750 2600
-F 0 "#FLG0101" H 750 2675 50  0001 C CNN
+F 0 "#FLG03" H 750 2675 50  0001 C CNN
 F 1 "PWR_FLAG" H 750 2774 50  0000 C CNN
 F 2 "" H 750 2600 50  0001 C CNN
@@
 $EndComp
 $Comp
-L KLIB_Power:PWR_FLAG #FLG0102
-U 1 1 5AE70EFD
+L KLIB_Power:PWR_FLAG #FLG04
+U 1 1 5AD7FB3D
 P 1250 2600
-F 0 "#FLG0102" H 1250 2675 50  0001 C CNN
+F 0 "#FLG04" H 1250 2675 50  0001 C CNN
 F 1 "PWR_FLAG" H 1250 2774 50  0000 C CNN
 F 2 "" H 1250 2600 50  0001 C CNN

Commit message: updated schematic added footptints
Parts:
- C18, C19, C20, C21, C22, C23, C24, C25: footprint (none) -> Capacitor_SMD:C_0805_2012Metric
- R13, R14: footprint (none) -> Resistor_SMD:R_0805_2012Metric
- U7: footprint LQFP64 -> Package_QFP:TQFP-64_10x10mm_P0.5mm
Changed lines of the file:
@@
 F 0 "U7" H 1650 5850 50  0000 L CNN
 F 1 "STM32F405RGTx" H 1650 5750 50  0000 L CNN
-F 2 "LQFP64" H 10050 5625 50  0001 R TNN
+F 2 "Package_QFP:TQFP-64_10x10mm_P0.5mm" H 10050 5625 50  0001 R TNN
 F 3 "http://www.st.com/st-web-ui/static/active/en/resource/technical/document/datasheet/DM00037051.pdf" H 5850 3750 50  0001 C CNN
 	1    5850 3750
@@
 F 0 "R14" H 1170 1996 50  0000 L CNN
 F 1 "10k" H 1170 1905 50  0000 L CNN
-F 2 "" V 1030 1950 50  0001 C CNN
+F 2 "Resistor_SMD:R_0805_2012Metric" V 1030 1950 50  0001 C CNN
 F 3 "~" H 1100 1950 50  0001 C CNN
 	1    1100 1950
@@
 F 0 "R13" H 820 1996 50  0000 L CNN
 F 1 "10k" H 820 1905 50  0000 L CNN
-F 2 "" V 680 1950 50  0001 C CNN
+F 2 "Resistor_SMD:R_0805_2012Metric" V 680 1950 50  0001 C CNN
 F 3 "~" H 750 1950 50  0001 C CNN
 	1    750  1950
@@
 F 0 "C18" H 865 2996 50  0000 L CNN
 F 1 "100n" H 865 2905 50  0000 L CNN
-F 2 "" H 788 2800 50  0001 C CNN
+F 2 "Capacitor_SMD:C_0805_2012Metric" H 788 2800 50  0001 C CNN
 F 3 "~" H 750 2950 50  0001 C CNN
 	1    750  2950
@@
 F 0 "C19" H 1365 2996 50  0000 L CNN
 F 1 "100n" H 1365 2905 50  0000 L CNN
-F 2 "" H 1288 2800 50  0001 C CNN
+F 2 "Capacitor_SMD:C_0805_2012Metric" H 1288 2800 50  0001 C CNN
 F 3 "~" H 1250 2950 50  0001 C CNN
 	1    1250 2950
@@
 F 0 "C21" H 7865 1196 50  0000 L CNN
 F 1 "100n" H 7865 1105 50  0000 L CNN
-F 2 "" H 7788 1000 50  0001 C CNN
+F 2 "Capacitor_SMD:C_0805_2012Metric" H 7788 1000 50  0001 C CNN
 F 3 "~" H 7750 1150 50  0001 C CNN
 	1    7750 1150
@@
 F 0 "C22" H 8315 1196 50  0000 L CNN
 F 1 "100n" H 8315 1105 50  0000 L CNN
-F 2 "" H 8238 1000 50  0001 C CNN
+F 2 "Capacitor_SMD:C_0805_2012Metric" H 8238 1000 50  0001 C CNN
 F 3 "~" H 8200 1150 50  0001 C CNN
 	1    8200 1150
@@
 F 0 "C23" H 8765 1196 50  0000 L CNN
 F 1 "100n" H 8765 1105 50  0000 L CNN
-F 2 "" H 8688 1000 50  0001 C CNN
+F 2 "Capacitor_SMD:C_0805_2012Metric" H 8688 1000 50  0001 C CNN
 F 3 "~" H 8650 1150 50  0001 C CNN
 	1    8650 1150
@@
 F 0 "C24" H 9215 1196 50  0000 L CNN
 F 1 "100n" H 9215 1105 50  0000 L CNN
-F 2 "" H 9138 1000 50  0001 C CNN
+F 2 "Capacitor_SMD:C_0805_2012Metric" H 9138 1000 50  0001 C CNN
 F 3 "~" H 9100 1150 50  0001 C CNN
 	1    9100 1150
@@
 F 0 "C25" H 9665 1196 50  0000 L CNN
 F 1 "100n" H 9665 1105 50  0000 L CNN
-F 2 "" H 9588 1000 50  0001 C CNN
+F 2 "Capacitor_SMD:C_0805_2012Metric" H 9588 1000 50  0001 C CNN
 F 3 "~" H 9550 1150 50  0001 C CNN
 	1    9550 1150
@@
 F 0 "C20" H 7415 1196 50  0000 L CNN
 F 1 "100n" H 7415 1105 50  0000 L CNN
-F 2 "" H 7338 1000 50  0001 C CNN
+F 2 "Capacitor_SMD:C_0805_2012Metric" H 7338 1000 50  0001 C CNN
 F 3 "~" H 7300 1150 50  0001 C CNN
 	1    7300 1150

Commit message: updated schematic
Parts:
- renumbered U7 to U6
Changed lines of the file:
@@
 $EndDescr
 $Comp
-L MCU_ST_STM32:STM32F405RGTx U7
+L MCU_ST_STM32:STM32F405RGTx U6
 U 1 1 5AD7FB27
 P 5850 3750
-F 0 "U7" H 1650 5850 50  0000 L CNN
+F 0 "U6" H 1650 5850 50  0000 L CNN
 F 1 "STM32F405RGTx" H 1650 5750 50  0000 L CNN
 F 2 "Package_QFP:TQFP-64_10x10mm_P0.5mm" H 10050 5625 50  0001 R TNN

Commit message: updated pcb
Connections:
- net SOUND_SEL0: now also U6.44 (ADC1_EXTI11/ADC2_EXTI11/ADC3_EXTI11/CAN1_RX/TIM1_CH4/USART1_CTS/USB_OTG_FS_DM/PA11); no longer U6.14 (ADC1_IN0/ADC2_IN0/ADC3_IN0/SYS_WKUP/TIM2_CH1/TIM2_ETR/TIM5_CH1/TIM8_ETR/UART4_TX/USART2_CTS/PA0)
- net SOUND_SEL1: now also U6.45 (CAN1_TX/TIM1_ETR/USART1_RTS/USB_OTG_FS_DP/PA12); no longer U6.15 (ADC1_IN1/ADC2_IN1/ADC3_IN1/TIM2_CH2/TIM5_CH2/UART4_RX/USART2_RTS/PA1)
Changed lines of the file:
@@
 NoConn ~ 10150 4850
 NoConn ~ 10150 4950
-NoConn ~ 10150 3250
-NoConn ~ 10150 3350
 NoConn ~ 10150 3950
 NoConn ~ 10150 3850
@@
 DAC
 Wire Wire Line
-	10150 2150 10400 2150
+	10150 3250 10400 3250
 Wire Wire Line
-	10150 2250 10400 2250
-Text HLabel 10400 2150 2    50   Input ~ 0
+	10150 3350 10400 3350
+Text HLabel 10400 3250 2    50   Input ~ 0
 SOUND_SEL0
-Text HLabel 10400 2250 2    50   Input ~ 0
+Text HLabel 10400 3350 2    50   Input ~ 0
 SOUND_SEL1
 Wire Wire Line
@@
 	1    0    0    -1
 $EndComp
+NoConn ~ 10150 2150
+NoConn ~ 10150 2250
 $EndSCHEMATC
