File: hw/main.kicad_pcb (KiCad board)
At the start: 2 copper layers, 110 x 85 mm, 106 parts, among them J1 UART_01X03, J2 SWD_01X04, J3 SWD_01X04, J4 IDC_02X07, J5 IDC_02X07, J6 IDC_02X03, J7 IDC_02X13, J8 SMA, J9 IDC_02X05, SW1 LCD_BTN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

Commit message: updated pcb
Routing:
- net /Display/LCD_UART_RX: track 0.00 -> 101.2 mm, vias 0 -> 1
- net /Display/~LCD_RST: track 0.00 -> 98.7 mm, vias 0 -> 1
- net /Main MCU/LCD_UART_RX: track 0.00 -> 96.8 mm, vias 0 -> 1
- net +5V: track 32.7 -> 50.8 mm
Changed lines of the file:
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@@
     (thickness 1.6)
     (drawings 7)
-    (tracks 348)
+    (tracks 410)
     (zones 0)
     (modules 106)
@@
   )
   (setup
-    (last_trace_width 1)
+    (last_trace_width 0.25)
     (user_trace_width 0.5)
     (user_trace_width 0.8)
@@
   (segment (start 182.6 81.7) (end 180.18 81.7) (width 0.5) (layer F.Cu) (net 10))
   (segment (start 180.18 81.7) (end 179.88 82) (width 0.5) (layer F.Cu) (net 10))
+  (segment (start 109.16 51) (end 109.16 55.59) (width 1) (layer F.Cu) (net 13))
+  (segment (start 109.16 55.59) (end 106.25 58.5) (width 1) (layer F.Cu) (net 13))
+  (segment (start 106.25 58.5) (end 106.25 67.9) (width 1) (layer F.Cu) (net 13))
+  (segment (start 104 67.9) (end 106.25 67.9) (width 1) (layer F.Cu) (net 13))
+  (segment (start 106.25 67.9) (end 108.5 67.9) (width 1) (layer F.Cu) (net 13))
   (segment (start 110.75 67.9) (end 112.944252 67.9) (width 1) (layer F.Cu) (net 13))
   (segment (start 108.5 67.9) (end 110.75 67.9) (width 1) (layer F.Cu) (net 13))
@@
   (segment (start 110.5 67.65) (end 110.5 65.63) (width 1) (layer F.Cu) (net 13))
   (segment (start 108.5 67.9) (end 108.5 65.63) (width 1) (layer F.Cu) (net 13))
-  (segment (start 104 67.9) (end 108.5 67.9) (width 1) (layer F.Cu) (net 13))
   (segment (start 102 67.9) (end 104 67.9) (width 1) (layer F.Cu) (net 13))
   (segment (start 104 67.9) (end 104 65.63) (width 1) (layer F.Cu) (net 13))
@@
   (segment (start 170.5 84) (end 175 88.5) (width 0.25) (layer F.Cu) (net 63))
   (segment (start 175 88.5) (end 175 93.797919) (width 0.25) (layer F.Cu) (net 63))
-  (segment (start 103.8 99.5) (end 97.5 99.5) (width 0.25) (layer F.Cu) (net 76))
-  (segment (start 97.5 99.5) (end 95 97) (width 0.25) (layer F.Cu) (net 76))
+  (segment (start 100.5 101.75) (end 100 101.25) (width 0.25) (layer B.Cu) (net 72))
+  (segment (start 100 100.5) (end 100.274999 100.225001) (width 0.25) (layer B.Cu) (net 72))
+  (segment (start 100.598001 100.225001) (end 100.975001 99.848001) (width 0.25) (layer B.Cu) (net 72))
+  (segment (start 100 101.25) (end 100 100.5) (width 0.25) (layer B.Cu) (net 72))
+  (segment (start 100.975001 99.848001) (end 100.975001 99.151999) (width 0.25) (layer B.Cu) (net 72))
+  (segment (start 129.200011 51.686398) (end 138.58642 42.299989) (width 0.25) (layer B.Cu) (net 72))
+  (segment (start 100.274999 100.225001) (end 100.598001 100.225001) (width 0.25) (layer B.Cu) (net 72))
+  (segment (start 100.975001 99.151999) (end 100.740757 98.917755) (width 0.25) (layer B.Cu) (net 72))
+  (segment (start 138.58642 42.299989) (end 142.950011 42.299989) (width 0.25) (layer B.Cu) (net 72))
+  (segment (start 143.5 41.75) (end 143.5 39.96) (width 0.25) (layer B.Cu) (net 72))
+  (segment (start 144.136401 39.323599) (end 145 38.46) (width 0.25) (layer B.Cu) (net 72))
+  (segment (start 143.5 39.96) (end 144.136401 39.323599) (width 0.25) (layer B.Cu) (net 72))
+  (segment (start 129.200011 67.4364) (end 129.200011 51.686398) (width 0.25) (layer B.Cu) (net 72))
+  (segment (start 105.5636 73.549989) (end 123.086422 73.549989) (width 0.25) (layer B.Cu) (net 72))
+  (segment (start 123.086422 73.549989) (end 129.200011 67.4364) (width 0.25) (layer B.Cu) (net 72))
+  (segment (start 101.75 101.75) (end 100.5 101.75) (width 0.25) (layer B.Cu) (net 72))
+  (segment (start 100.740757 98.917755) (end 100.740757 78.372832) (width 0.25) (layer B.Cu) (net 72))
+  (segment (start 100.740757 78.372832) (end 105.5636 73.549989) (width 0.25) (layer B.Cu) (net 72))
+  (segment (start 142.950011 42.299989) (end 143.5 41.75) (width 0.25) (layer B.Cu) (net 72))
+  (segment (start 102 101.5) (end 101.75 101.75) (width 0.25) (layer F.Cu) (net 72))
+  (segment (start 103.8 101.5) (end 102 101.5) (width 0.25) (layer F.Cu) (net 72))
+  (via (at 101.75 101.75) (size 0.8) (drill 0.4) (layers F.Cu B.Cu) (net 72))
+  (segment (start 129.650022 51.872798) (end 138.77282 42.75) (width 0.25) (layer B.Cu) (net 73))
+  (segment (start 123.272822 74) (end 129.650022 67.6228) (width 0.25) (layer B.Cu) (net 73))
+  (segment (start 101.190768 98.731355) (end 101.190768 78.559232) (width 0.25) (layer B.Cu) (net 73))
+  (segment (start 100.828776 100.912302) (end 101.425012 100.316066) (width 0.25) (layer B.Cu) (net 73))
+  (segment (start 129.650022 67.6228) (end 129.650022 51.872798) (width 0.25) (layer B.Cu) (net 73))
+  (segment (start 101.425012 98.965599) (end 101.190768 98.731355) (width 0.25) (layer B.Cu) (net 73))
+  (segment (start 145.79 42.75) (end 146.676401 41.863599) (width 0.25) (layer B.Cu) (net 73))
+  (segment (start 101.425012 100.316066) (end 101.425012 98.965599) (width 0.25) (layer B.Cu) (net 73))
+  (segment (start 101.190768 78.559232) (end 105.75 74) (width 0.25) (layer B.Cu) (net 73))
+  (segment (start 146.676401 41.863599) (end 147.54 41) (width 0.25) (layer B.Cu) (net 73))
+  (segment (start 105.75 74) (end 123.272822 74) (width 0.25) (layer B.Cu) (net 73))
+  (segment (start 138.77282 42.75) (end 145.79 42.75) (width 0.25) (layer B.Cu) (net 73))
+  (via (at 100.828776 100.912302) (size 0.8) (drill 0.4) (layers F.Cu B.Cu) (net 73))
+  (segment (start 103.8 101) (end 100.916474 101) (width 0.25) (layer F.Cu) (net 73))
+  (segment (start 100.916474 101) (end 100.828776 100.912302) (width 0.25) (layer F.Cu) (net 73))
+  (segment (start 122.900022 73.099978) (end 128.75 67.25) (width 0.25) (layer B.Cu) (net 74))
+  (segment (start 128.75 51.499998) (end 138.40002 41.849978) (width 0.25) (layer B.Cu) (net 74))
+  (segment (start 100.25 78.227178) (end 105.3772 73.099978) (width 0.25) (layer B.Cu) (net 74))
+  (segment (start 143 41.5) (end 143 38.5) (width 0.25) (layer B.Cu) (net 74))
+  (segment (start 146.08 37) (end 146.676401 37.596401) (width 0.25) (layer B.Cu) (net 74))
+  (segment (start 100.25 99.5) (end 100.25 78.227178) (width 0.25) (layer B.Cu) (net 74))
+  (segment (start 138.40002 41.849978) (end 142.650022 41.849978) (width 0.25) (layer B.Cu) (net 74))
+  (segment (start 143 38.5) (end 144.5 37) (width 0.25) (layer B.Cu) (net 74))
+  (segment (start 128.75 67.25) (end 128.75 51.499998) (width 0.25) (layer B.Cu) (net 74))
+  (segment (start 144.5 37) (end 146.08 37) (width 0.25) (layer B.Cu) (net 74))
+  (segment (start 105.3772 73.099978) (end 122.900022 73.099978) (width 0.25) (layer B.Cu) (net 74))
+  (segment (start 146.676401 37.596401) (end 147.54 38.46) (width 0.25) (layer B.Cu) (net 74))
+  (segment (start 142.650022 41.849978) (end 143 41.5) (width 0.25) (layer B.Cu) (net 74))
+  (segment (start 100.973001 99.899999) (end 100.649999 99.899999) (width 0.25) (layer F.Cu) (net 74))
+  (segment (start 101.573002 100.5) (end 100.973001 99.899999) (width 0.25) (layer F.Cu) (net 74))
+  (segment (start 103.8 100.5) (end 101.573002 100.5) (width 0.25) (layer F.Cu) (net 74))
+  (segment (start 100.649999 99.899999) (end 100.25 99.5) (width 0.25) (layer F.Cu) (net 74))
+  (via (at 100.25 99.5) (size 0.8) (drill 0.4) (layers F.Cu B.Cu) (net 74))
+  (segment (start 95 92) (end 96.150001 90.849999) (width 0.25) (layer F.Cu) (net 76))
+  (segment (start 103.8 99.5) (end 102.8 99.5) (width 0.25) (layer F.Cu) (net 76))
+  (segment (start 96.150001 90.849999) (end 97 90) (width 0.25) (layer F.Cu) (net 76))
+  (segment (start 101.931413 98.631413) (end 96.631413 98.631413) (width 0.25) (layer F.Cu) (net 76))
   (segment (start 95 97) (end 95 92) (width 0.25) (layer F.Cu) (net 76))
-  (segment (start 95 92) (end 97 90) (width 0.25) (layer F.Cu) (net 76))
+  (segment (start 96.631413 98.631413) (end 95 97) (width 0.25) (layer F.Cu) (net 76))
+  (segment (start 102.8 99.5) (end 101.931413 98.631413) (width 0.25) (layer F.Cu) (net 76))
   (segment (start 106.25 97.55) (end 106.25 94.5) (width 0.25) (layer F.Cu) (net 77))
   (segment (start 106.25 94.5) (end 105.25 93.5) (width 0.25) (layer F.Cu) (net 77))

Commit message: updated pcb
Parts:
- moved C4 1.00 mm to (100.0, 108.2)
- moved R1 1.00 mm to (100.0, 106.2)
Routing:
- net /Back/~INT: track 0.00 -> 79.0 mm, vias 0 -> 1
- net /Back/SDA: track 0.00 -> 8.38 mm, vias 0 -> 1
- net /Back/SCL: track 0.00 -> 7.73 mm, vias 0 -> 1
- net /Back/~AL: track 0.00 -> 7.09 mm, vias 0 -> 1
- net Net-(R1-Pad2): track 3.02 -> 3.73 mm
- net +3V3: track 44.7 -> 45.4 mm
