File: hw/main.kicad_pcb (KiCad board)
At the start: 2 copper layers, 110 x 85 mm, 106 parts, among them J1 UART_01X03, J2 SWD_01X04, J3 SWD_01X04, J4 IDC_02X07, J5 IDC_02X07, J6 IDC_02X03, J7 IDC_02X13, J8 SMA, J9 IDC_02X05, SW1 LCD_BTN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

Commit message: updated pcb
Routing:
- net /Back/~AL: track 7.09 -> 81.6 mm
- net /Back/SDA: track 8.38 -> 82.0 mm
- net /Back/SCL: track 7.73 -> 81.3 mm

Commit message: updated pcb
Parts:
- moved C17 4.03 mm to (177.8, 55.0), turned to 90 degrees
- moved C13 4.00 mm to (186.2, 55.0)
- moved R11 4.00 mm to (190.2, 55.0)
- moved R2 3.76 mm to (100.0, 94.5), turned to 90 degrees
- moved R10 2.25 mm to (188.8, 64.0)
- moved R3 2.12 mm to (155.0, 59.0)
- moved R7 2.12 mm to (170.2, 59.0)
- moved C11 2.00 mm to (186.5, 64.0)
- moved C9 0.25 mm to (153.0, 59.0)
- moved R9 0.25 mm to (188.8, 70.0)
- turned R8 to 270 degrees
Routing:
- net /Shoulder 1/SPEAKER+: track 0.00 -> 45.1 mm
- net /Sound/MUTE: track 0.00 -> 42.6 mm, vias 0 -> 3
- net /Shoulder 1/SPEAKER-: track 0.00 -> 41.1 mm
- net /Main MCU/~RST: track 0.00 -> 39.2 mm, vias 0 -> 1
- net /Shoulder 2/SPEAKER-: track 0.00 -> 29.3 mm, vias 0 -> 1
- net Net-(C17-Pad1): track 0.00 -> 28.7 mm
- net Net-(C12-Pad2): track 0.00 -> 22.6 mm
- net /Shoulder 2/SPEAKER+: track 0.00 -> 20.9 mm
- net Net-(C15-Pad2): track 0.00 -> 12.1 mm
- net Net-(R9-Pad2): track 0.00 -> 11.0 mm
- net Net-(C17-Pad2): track 0.00 -> 9.27 mm
- net Net-(C15-Pad1): track 0.00 -> 9.03 mm
- net Net-(C13-Pad1): track 0.00 -> 8.85 mm
- net Net-(R7-Pad1): track 0.00 -> 7.62 mm
- net Net-(R3-Pad1): track 0.00 -> 7.62 mm
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
Commit message: updated pcb
Parts:
- moved C35 4.83 mm to (141.2, 83.8), turned to 180 degrees
- moved R27 0.93 mm to (145.2, 77.0)
Routing:
- net +5V: track 50.8 -> 315.1 mm, vias 0 -> 7
- net Net-(C35-Pad1): track 0.00 -> 8.07 mm

Commit message: updated pcb
Routing:
- net /Back/LED_PWM_R: track 0.00 -> 163.9 mm, vias 0 -> 3
- net /Back/LED_PWM_G: track 0.00 -> 156.9 mm, vias 0 -> 4
- net /Back/LED_PWM_B: track 0.00 -> 150.2 mm, vias 0 -> 4
- net /Display/~LCD_RST: track 98.7 -> 95.5 mm
- net /Main MCU/LCD_UART_RX: track 96.7 -> 93.5 mm
- net /Display/LCD_UART_RX: track 101.0 -> 97.9 mm

Commit message: updated pcb
Parts:
- moved C26 0.20 mm to (99.0, 112.8)
- moved SW1 0.20 mm to (96.0, 112.8)
Connections:
- J7 pad 11: GND -> /Back/LED_PWM_R
- J7 pad 12: /Back/LED_PWM_R -> GND
- J7 pad 13: GND -> /Back/LED_PWM_G
- J7 pad 14: /Back/LED_PWM_G -> GND
- J7 pad 15: GND -> /Back/LED_PWM_B
- J7 pad 16: /Back/LED_PWM_B -> GND
- J7 pad 17: GND -> /Back/SDA
- J7 pad 18: /Back/SDA -> GND
- J7 pad 19: GND -> /Back/SCL
- J7 pad 20: /Back/SCL -> GND
- J7 pad 21: GND -> /Back/~INT
- J7 pad 22: /Back/~INT -> GND
- J7 pad 23: GND -> /Back/~AL
- J7 pad 24: /Back/~AL -> GND
- J7 pad 25: GND -> /Back/IR_RX
- J7 pad 26: /Back/IR_RX -> GND
Routing:
- net /Back/LED_PWM_B: track 150.2 -> 240.1 mm, vias 4 -> 7
- net /Back/IR_RX: track 2.54 -> 78.3 mm
- net /Back/LED_PWM_R: track 163.9 -> 237.8 mm, vias 3 -> 4
- net /Back/LED_PWM_G: track 156.9 -> 224.6 mm, vias 4 -> 7
- net /Gun/GUN_RX: track 2.54 -> 67.1 mm, vias 0 -> 1
- net /Gun/GUN_TX: track 2.54 -> 55.9 mm, vias 0 -> 1
- net /Back/~AL: track 81.6 -> 79.1 mm
- net /Back/~INT: track 78.7 -> 76.2 mm
- net /Back/SCL: track 81.3 -> 78.8 mm
- net /Back/SDA: track 82.0 -> 79.4 mm
- net +5V5: track 110.9 -> 110.1 mm

Commit message: updated pcb
Parts:
- moved C36 1.25 mm to (165.8, 100.3)
- moved C37 1.25 mm to (165.8, 98.4)
Routing:
- net +3V3: track 45.4 -> 328.7 mm, vias 0 -> 29
- net /Back/IR_RX: track 78.3 -> 211.9 mm, vias 0 -> 2
- net Net-(R5-Pad2): track 0.00 -> 47.1 mm, vias 0 -> 2
- net /Shoulder 1/SPEAKER+: track 45.1 -> 48.3 mm
- net /Sound/Sound MCU/~RST: track 37.1 -> 34.7 mm
- net /Sound/Sound MCU/SWDCLK: track 15.4 -> 16.6 mm, vias 0 -> 1
- net +5V: track 315.1 -> 313.9 mm
- net /Back/LED_PWM_R: track 237.8 -> 238.8 mm

Commit message: updated pcb
Parts:
- moved C18 0.50 mm to (152.5, 82.0)
- moved C22 0.50 mm to (152.5, 84.0)
- moved C25 0.50 mm to (152.5, 77.5)
- moved R5 0.50 mm to (152.5, 79.5)
- moved R6 0.50 mm to (152.5, 75.5)
Routing:
- net GND: track 0.00 -> 11.2 mm, vias 0 -> 44
- net Net-(R5-Pad2): track 47.1 -> 51.2 mm
- net +3V3: track 328.7 -> 332.4 mm, vias 29 -> 30
- net /Main MCU/SWDIO: track 16.9 -> 17.6 mm
- net +5V: track 313.9 -> 313.4 mm
- net Net-(C18-Pad1): track 3.70 -> 4.20 mm

Commit message: updated pcb
Routing:
- net /Back/IR_RX: track 211.9 -> 206.9 mm
- net /Display/~LCD_RST: track 95.5 -> 90.9 mm
- net /Main MCU/LCD_UART_RX: track 93.5 -> 88.9 mm
- net /Display/LCD_UART_RX: track 97.9 -> 93.3 mm
- net /Back/LED_PWM_B: track 240.1 -> 238.5 mm
- net /Back/LED_PWM_G: track 224.6 -> 225.5 mm
- net GND: vias 44 -> 74
